Commit message: chapt7_ws/src/fishbot_navigation2/ : build map, v01

File: chapt7_ws/src/fishbot_description/urdf/fishbot/actuator/wheel.urdf.xacro (robot description, xacro)
@@ -13,8 +13,15 @@
                 </material>
             </visual>
+            <!--
+              碰撞体用球体而不是圆柱体：圆柱轮与地面接触时，ODE 会把接触点
+              放在圆柱两端的棱边上，等效轮距会在 0.16 m（内棱）和 0.24 m（外棱）
+              之间跳变，导致里程计偏航角出现 ±20% 的随机误差，SLAM 建图会重影。
+              球体的接触点固定在轮子中心正下方（y=±0.10 m），与 wheel_separation
+              参数一致。视觉仍保留圆柱体，外观不变。
+            -->
             <collision>
-                <origin xyz="0 0 0" rpy="1.57079 0 0" />
+                <origin xyz="0 0 0" rpy="0 0 0" />
                 <geometry>
-                    <cylinder length="0.04" radius="0.032" />
+                    <sphere radius="0.032" />
                 </geometry>
                 <material name="black">

File: chapt7_ws/src/fishbot_description/urdf/fishbot/fishbot.ros2_control.xacro (robot description, xacro)
@@ -40,6 +40,11 @@
                 <parameters>$(find fishbot_description)/config/fishbot_ros2_controller.yaml</parameters>
                 <ros>
-                    <remapping>/fishbot_diff_drive_controller/cmd_vel:=/cmd_vel_01by_ros2control</remapping>
-                    <remapping>/fishbot_diff_drive_controller/odom:=/odom_01by_ros2control</remapping>
+                    <!-- 命名映射:
+                        原名称:=新名称
+                    -->
+                    <!-- ros2control订阅的话题 /cmd_vel -->
+                    <remapping>/fishbot_diff_drive_controller/cmd_vel:=/cmd_vel</remapping>
+                    <!-- ros2control发布的话题 /odom -->
+                    <remapping>/fishbot_diff_drive_controller/odom:=/odom</remapping>
                 </ros>
             </plugin>

File: chapt7_ws/src/fishbot_description/urdf/fishbot/plugins/gazebo_control_plugin.xacro (robot description, xacro)
@@ -17,4 +17,5 @@
     <robot_base_frame>base_footprint</robot_base_frame>
     <!-- 话题名称（Harmonic DiffDrive插件原生发布gz消息，需要ros_gz_bridge转ROS2话题） -->
+    <!-- 订阅话题/cmd_vel ； 发布话题 /gz/odom  -->
     <cmd_vel_topic>/cmd_vel_00by_diff_drive</cmd_vel_topic>
     <odom_topic>/gz/odom_00by_diff_drive</odom_topic>

File: chapt7_ws/src/fishbot_description/urdf/fishbot/plugins/gazebo_sensor_plugin.xacro (robot description, xacro)
@@ -10,5 +10,5 @@
                 <update_rate>10</update_rate>
                 <pose>0 0 0 0 0 0</pose>
-                <topic>/scan1</topic>
+                <topic>/scan</topic>
                 <gz_frame_id>laser_link</gz_frame_id>
 				<!-- 激光传感器配置 -->
@@ -26,5 +26,9 @@
                     <range>
                         <min>0.120000</min>
-                        <max>8.0</max>
+                        <!-- 房子约 19 x 11 m（对角线约 22 m）。原来 8.0 m 在大厅和
+                             长走廊里大量打空，而无回波的返回值就是 <max>，会和真实
+                             最远读数混在一起。25.0 留出余量，与 slam_toolbox 的
+                             max_laser_range: 23.0 配套使用。 -->
+                        <max>25.0</max>
                         <resolution>0.015000</resolution>
                     </range>
